Commit message: modified UI code and move_base paramters

File: demconRobot.xacro (robot description, xacro)
@@ -3,7 +3,7 @@
 	<xacro:property name="bodyWidth" value="0.36" />
 	<xacro:property name="bodyLength" value="0.44" />
-	<xacro:property name="bodyHeigth" value="0.054" />
-	<xacro:property name="wheelRadius" value="0.0825" />
-	<xacro:property name="wheelWidth" value="0.092" />
+	<xacro:property name="bodyHeigth" value="0.055" />
+	<xacro:property name="wheelRadius" value="0.085" />
+	<xacro:property name="wheelWidth" value="0.098" />
 	<xacro:property name="M_PI" value="3.1415926535" />
 	<link name="base_footprint">
@@ -13,4 +13,8 @@
 			</geometry>
 		</visual>
+		<collision>
+			<geometry>
+			</geometry>
+		</collision>
 	</link>
 	<link name="base_link">
@@ -23,9 +27,9 @@
 			</material>
 		</visual>
-		<collision>
+		<!--<collision>
 			<geometry>
 				<cylinder length="0.2" radius="0.4" />
 			</geometry>
-		</collision>
+		</collision>-->
 	</link>
 	<joint name="base_footprint_joint" type="fixed">
@@ -76,5 +80,5 @@
 			<origin rpy="0 0 0" xyz="0 0 ${wheelRadius}"/>
 			<geometry>
-				<cylinder radius="0.03" length="0.01" />
+				<cylinder radius="0.033" length="0.01" />
 			</geometry>
 			<material name="white">
@@ -116,5 +120,5 @@
 		<parent link="base_link"/>
 		<child link="laser_scanner"/>
-		<origin xyz="0 0.18 0" rpy="0 0 ${-0.5*M_PI}"/>
+		<origin xyz="0 0.185 0" rpy="0 0 ${-0.5*M_PI}"/>
 	</joint>
 	<joint name="base_to_imu" type="fixed">

Commit message: added comments and removed old code

File: demconRobot.xacro (robot description, xacro)
@@ -13,8 +13,4 @@
 			</geometry>
 		</visual>
-		<collision>
-			<geometry>
-			</geometry>
-		</collision>
 	</link>
 	<link name="base_link">
@@ -27,9 +23,4 @@
 			</material>
 		</visual>
-		<!--<collision>
-			<geometry>
-				<cylinder length="0.2" radius="0.4" />
-			</geometry>
-		</collision>-->
 	</link>
 	<joint name="base_footprint_joint" type="fixed">
@@ -78,5 +69,5 @@
 	<link name="laser_scanner">
 		<visual>
-			<origin rpy="0 0 0" xyz="0 0 ${wheelRadius}"/>
+			<origin rpy="0 0 0" xyz="0 0 0.1"/>
 			<geometry>
 				<cylinder radius="0.033" length="0.01" />
@@ -125,5 +116,5 @@
 		<parent link="base_link"/>
 		<child link="base_imu"/>
-		<origin xyz="0 0 0.001" rpy="0 0 0"/>
+		<origin xyz="0 0 0" rpy="0 0 0"/>
 	</joint>
 </robot>
